Commit message: adding leaf remover link

File: denso_robot_descriptions/vs060_description/vs060.urdf (robot description, URDF)
Before this commit: robot vs060, 8 links, 7 joints
Links:
- added link leaf_remover_base_link, mass 0.1; collision mesh filename=package://denso_robot_descriptions/vs060_description/leaf_r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 scale=0.001 0.001 0.001; visual mesh filename=package://denso_robot_descriptions/vs060_description/leaf_r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 scale=0.001 0.001 0.001
Joints:
- added joint leaf_remover_joint: type fixed, parent J6, child leaf_remover_base_link, origin xyz=0 0 0 rpy=0 0 0

Commit message: added leaf remover to the robot model

File: denso_robot_descriptions/vs060_description/vs060.urdf (robot description, URDF)
Before this commit: robot vs060, 9 links, 8 joints
Links:
- added link leaf_remover_first_link, mass 0.1; collision box size=0.04 0.029 0.028; visual box size=0.04 0.029 0.028
- added link leaf_remover_second_link, mass 0.1; collision box size=0.04 0.088 0.028; visual box size=0.04 0.196 0.028
- link leaf_remover_base_link: mass 0.1 -> 0.4; geometry collision box size=0.04 0.0587 0.25; visual box size=0.04 0.0587 0.25
Joints:
- added joint leaf_remover_joint_1: type fixed, parent leaf_remover_base_link, child leaf_remover_first_link, origin xyz=0.0 0.04385 0.125 rpy=0 30 0
- added joint leaf_remover_joint_2: type fixed, parent leaf_remover_first_link, child leaf_remover_second_link, origin xyz=0.0 0.1025 0.0 rpy=0 0 0
- joint leaf_remover_joint: origin xyz=0 0 0 rpy=0 0 0 -> xyz=0 0 0.125 rpy=0 0 0

Commit message: added start pose

File: denso_robot_descriptions/vs060_description/vs060.urdf (robot description, URDF)
Before this commit: robot vs060, 11 links, 10 joints
Joints:
- joint leaf_remover_joint_1: origin xyz=0.0 0.04385 0.125 rpy=0 30 0 -> xyz=0.0 0.04385 0.125 rpy=0 0 0

Commit message: changed robot model

File: denso_robot_descriptions/vs060_description/vs060.urdf (robot description, URDF)
Before this commit: robot vs060, 11 links, 10 joints
Joints:
- joint leaf_remover_joint: origin xyz=0 0 0.125 rpy=0 0 0 -> xyz=0 0 0.25 rpy=0 0 0
- joint leaf_remover_joint_1: origin xyz=0.0 0.04385 0.125 rpy=0 0 0 -> xyz=0.0 0.05835 0.0   rpy=0 0 0
- joint leaf_remover_joint_2: origin xyz=0.0 0.1025 0.0 rpy=0 0 0 -> xyz=0.0 0.196 0.0 rpy=0 0 0

Commit message: revised the model and start pose

File: denso_robot_descriptions/vs060_description/vs060.urdf (robot description, URDF)
Before this commit: robot vs060, 11 links, 10 joints
Links:
- link leaf_remover_base_link: geometry collision box size=0.04 0.0587 0.35; visual box size=0.04 0.0587 0.35
Joints:
- joint leaf_remover_joint: origin xyz=0 0 0.25 rpy=0 0 0 -> xyz=0 0 0.35 rpy=0 0 0

Commit message: modifying model

File: denso_robot_descriptions/vs060_description/vs060.urdf (robot description, URDF)
Before this commit: robot vs060, 11 links, 10 joints
Links:
- added link leaf_remover_third_link, mass 0.1; collision box size=0.04 0.088 0.028; visual box size=0.04 0.196 0.028
- link leaf_remover_base_link: geometry collision box size=0.04 0.1057 0.35; visual box size=0.04 0.1057 0.005
- link leaf_remover_first_link: mass 0.1 -> 0.4; geometry collision box size=0.04 0.04 0.345; visual box size=0.04 0.04 0.345
- link leaf_remover_second_link: geometry collision box size=0.04 0.0207 0.028; visual box size=0.04 0.0207 0.028
Joints:
- removed joint leaf_remover_joint
- added joint leaf_remover_joint_3: type fixed, parent leaf_remover_first_link, child leaf_remover_second_link, origin xyz=0.0 0.0407 0.0   rpy=0 0 0
- added joint leaf_remover_joint_4: type fixed, parent leaf_remover_second_link, child leaf_remover_third_link, origin xyz=0.0 0.196 0.0 rpy=0 0 0
- joint leaf_remover_joint_1: child leaf_remover_first_link -> leaf_remover_base_link; origin xyz=0.0 0.05835 0.0   rpy=0 0 0 -> xyz=0 -0.047 0.005 rpy=0 0 0; parent leaf_remover_base_link -> J6
- joint leaf_remover_joint_2: child leaf_remover_second_link -> leaf_remover_first_link; origin xyz=0.0 0.196 0.0 rpy=0 0 0 -> xyz=0 0 0.345 rpy=0 0 0; parent leaf_remover_first_link -> leaf_remover_base_link

Commit message: added zed to model

File: denso_robot_descriptions/vs060_description/vs060.urdf (robot description, URDF)
Before this commit: robot vs060, 12 links, 11 joints
Links:
- added link camera_mount; visual box size=0.02 0.120 0.014
Joints:
- added joint camera_mount_joint: type fixed, parent leaf_remover_base_link, child camera_mount, origin xyz=0 0.2525 0.014 rpy=0 0 0

Commit message: updated robot model

File: denso_robot_descriptions/vs060_description/vs060.urdf (robot description, URDF)
Before this commit: robot vs060, 13 links, 12 joints
Joints:
- joint leaf_remover_joint_1: origin xyz=0 -0.047 0.005 rpy=0 0 0 -> xyz=0 -0.06143 0.005 rpy=0 0 0

Commit message: modified for grape robot

File: denso_robot_descriptions/vs060_description/vs060.urdf (robot description, URDF)
Before this commit: robot vs060, 13 links, 12 joints
Joints:
- joint camera_mount_joint: origin xyz=0 0.2525 0.014 rpy=0 0 0 -> xyz=0 0.23 0.014 rpy=0 0 0

Commit message: changed frame and collision

File: denso_robot_descriptions/vs060_description/vs060.urdf (robot description, URDF)
Before this commit: robot vs060, 13 links, 12 joints
Joints:
- joint leaf_remover_joint_1: origin xyz=0 -0.06143 0.005 rpy=0 0 0 -> xyz=0 -0.06143 0.009 rpy=0 0 0
- joint leaf_remover_joint_2: origin xyz=0 0 0.345 rpy=0 0 0 -> xyz=0 0 0.341 rpy=0 0 0
